Commit message: "Archivos añadidos de práctica 1"

File: Prácticas/Práctica 1/robot_rrr_practicaV2.urdf (robot description, URDF)
Before this commit: robot robot, 5 links, 4 joints
Links:
- link arm_link: geometry 
- link base0_link: geometry 
- link base_link: geometry 
- link forearm_link: geometry 
- link shoulder_link: geometry 
Joints:
- joint arm_joint: limit lower=-3.14 upper=3.14 -> lower=-3.14 upper=3.14 effort=10 velocity=1
- joint base_joint: axis 0 0 0 -> (none); limit lower=0 upper=0 -> (none)
- joint forearm_joint: limit lower=-0.15 upper=0 -> lower=-0.15 upper=0 effort=10 velocity=1; origin xyz=0.3 0 0.35 rpy=1.57, 0, 0 -> xyz=0.3 0 0.35 rpy=1.57 0 0
- joint shoulder_joint: limit lower=-3.14 upper=3.14 -> lower=-3.14 upper=3.14 effort=10 velocity=1; origin (none) -> xyz=0 0 0.25
